Commit message: Updated geometry of robot, and got launch in Gazebo
Testing of differential drive plugin pending

File: swarm_ws/src/swarm_description/urdf/blackhawk_standalone.xacro (robot description, xacro)
@@ -1,24 +1,80 @@
 <?xml version="1.0"?>
-<robot name="blackhawk">
+<robot name="blackhawk" xmlns:xacro="http://ros.org/wiki/xacro">
   <link name="base_link">
+    <!-- Body geometry macro -->
+    <!-- <mesh filename="package://swarm_description/meshes/Blackhawk_resized.dae"/> -->
+    <xacro:property name="body_length" value="0.7"/>
+    <xacro:macro name="body">
+      <geometry>
+        <cylinder length="${body_length}" radius="0.5" />
+      </geometry>
+    </xacro:macro>
+    <xacro:property name="wheel_separation" value="0.2"/>
+    <xacro:property name="wheel_diameter" value="0.4"/>
+    <xacro:property name="wheel_width" value="0.05"/>
+    <!-- visual -->
     <visual>
-      <origin rpy="0.0 0 0" xyz="0 0 0"/>
-      <geometry>
-        <mesh filename="package://swarm_description/meshes/Blackhawk_resized.dae"/>
-      </geometry>
+	    <origin rpy="0.0 0 0" xyz="0 0 ${body_length / 2}"/>
+	    <xacro:body/>
     </visual>
-    <!-- TODO: add inertial & collision -->
+    <!-- inertial & collision -->
+    <collision>
+	    <origin rpy="0.0 0 0" xyz="0 0 ${body_length / 2}"/>
+        <xacro:body/>
+      </collision>
+    <inertial>
+      <mass value="0.5"/>
+      <inertia ixx="0.4" ixy="0.0" ixz="0.0" iyy="0.4" iyz="0.0" izz="0.2"/>
+    </inertial>
   </link>
-  <!-- TODO: Plugin to simulate driving motion -->
+  <!-- wheel joints -->
   <joint name="base_link_to_left_wheel" type="fixed">
     <child link="left_wheel" />
     <parent link="base_link" />
   </joint>
+  <joint name="base_link_to_right_wheel" type="fixed">
+	  <child link="right_wheel"/>
+	  <parent link="base_link"/>
+  </joint>
+  <!-- Wheel geometry macro -->
+  <xacro:macro name="wheel_geometry">
+    <geometry>
+	    <cylinder length="${wheel_width}" radius="${wheel_diameter / 2}"/>
+    </geometry>
+  </xacro:macro>
+  <!-- Wheel geometries -->
   <link name="left_wheel">
     <visual>
-      <origin rpy="0.0 0 0" xyz="0 0 0"/>
-      <geometry>
-      </geometry>
+      <origin rpy="0 1.57079 0" xyz="-${wheel_separation} 0 0"/>
+      <xacro:wheel_geometry/>
     </visual>
+    <collision>
+	    <origin rpy="0 1.57079 0" xyz="-${wheel_separation} 0 0"/>
+      <xacro:wheel_geometry/>
+    </collision>
   </link>
+  <link name="right_wheel">
+    <visual>
+      <origin rpy="0 -1.57079 0" xyz="${wheel_separation} 0 0"/>
+      <xacro:wheel_geometry/>
+    </visual>
+    <collision>
+	    <origin rpy="0 -1.57079 0" xyz="${wheel_separation} 0 0"/>
+      <xacro:wheel_geometry/>
+    </collision>
+  </link>
+  <!-- Plugin to simulate driving motion -->
+  <gazebo>
+    <plugin name="differential_drive_controller" filename="libgazebo_ros_diff_drive.so">
+      <alwaysOn>true</alwaysOn>
+      <updateRate>100</updateRate>
+      <leftJoint>base_link_to_left_wheel</leftJoint>
+      <rightJoint>base_link_to_right_wheel</rightJoint>
+      <wheelSeparation>${wheel_separation}</wheelSeparation>
+      <wheelDiameter>${wheel_diameter}</wheelDiameter>
+      <wheelTorque>2</wheelTorque>
+      <commandTopic>cmd_diff_vel</commandTopic>
+      <broadcastTF>false</broadcastTF>
+    </plugin>
+  </gazebo>
 </robot>

Commit message: Made dimensions realistic

File: swarm_ws/src/swarm_description/urdf/blackhawk_standalone.xacro (robot description, xacro)
@@ -4,13 +4,16 @@
     <!-- Body geometry macro -->
     <!-- <mesh filename="package://swarm_description/meshes/Blackhawk_resized.dae"/> -->
-    <xacro:property name="body_length" value="0.7"/>
+    <xacro:property name="body_length" value="0.06"/>
     <xacro:macro name="body">
       <geometry>
-        <cylinder length="${body_length}" radius="0.5" />
+        <!--<cylinder length="${body_length}" radius="0.5" /> -->
+        <mesh filename="package://swarm_description/meshes/Blackhawk_resized.dae"/>
       </geometry>
     </xacro:macro>
-    <xacro:property name="wheel_separation" value="0.2"/>
-    <xacro:property name="wheel_diameter" value="0.4"/>
-    <xacro:property name="wheel_width" value="0.05"/>
+    <!-- Values for different components of the robot-->
+    <xacro:property name="wheel_separation" value="0.02"/>
+    <xacro:property name="wheel_diameter" value="0.025"/>
+    <xacro:property name="wheel_width" value="0.005"/>
+    <xacro:property name="wheel_standoff" value="0.01"/>
     <!-- visual -->
     <visual>
@@ -24,6 +27,6 @@
       </collision>
     <inertial>
-      <mass value="0.5"/>
-      <inertia ixx="0.4" ixy="0.0" ixz="0.0" iyy="0.4" iyz="0.0" izz="0.2"/>
+      <mass value="0.2"/>
+      <inertia ixx="0.5" ixy="0.0" ixz="0.0" iyy="0.5" iyz="0.0" izz="0.5"/>
     </inertial>
   </link>
@@ -46,9 +49,9 @@
   <link name="left_wheel">
     <visual>
-      <origin rpy="0 1.57079 0" xyz="-${wheel_separation} 0 0"/>
+      <origin rpy="1.57079 0 0" xyz="${wheel_standoff} -${wheel_separation} 0"/>
       <xacro:wheel_geometry/>
     </visual>
     <collision>
-	    <origin rpy="0 1.57079 0" xyz="-${wheel_separation} 0 0"/>
+	    <origin rpy="1.57079 0 0" xyz="${wheel_standoff} -${wheel_separation} 0"/>
       <xacro:wheel_geometry/>
     </collision>
@@ -56,9 +59,9 @@
   <link name="right_wheel">
     <visual>
-      <origin rpy="0 -1.57079 0" xyz="${wheel_separation} 0 0"/>
+      <origin rpy="-1.57079 0 0" xyz="-${wheel_standoff} ${wheel_separation} 0"/>
       <xacro:wheel_geometry/>
     </visual>
     <collision>
-	    <origin rpy="0 -1.57079 0" xyz="${wheel_separation} 0 0"/>
+	    <origin rpy="-1.57079 0 0" xyz="-${wheel_standoff} ${wheel_separation} 0"/>
       <xacro:wheel_geometry/>
     </collision>

Commit message: Starting control of robot motion.

File: swarm_ws/src/swarm_description/urdf/blackhawk_standalone.xacro (robot description, xacro)
@@ -27,5 +27,5 @@
       </collision>
     <inertial>
-      <mass value="0.2"/>
+      <mass value="0.05"/>
       <inertia ixx="0.5" ixy="0.0" ixz="0.0" iyy="0.5" iyz="0.0" izz="0.5"/>
     </inertial>
@@ -69,15 +69,18 @@
   <!-- Plugin to simulate driving motion -->
   <gazebo>
-    <plugin name="differential_drive_controller" filename="libgazebo_ros_diff_drive.so">
+    <plugin name="gazebo_ros_control" filename="libgazebo_ros_control.so">
+      <robotSimType>gazebo_ros_control/DefaultRobotHWSim</robotSimType>
+    </plugin>
+    <!-- <plugin name="differential_drive_controller" filename="libgazebo_ros_diff_drive.so">
       <alwaysOn>true</alwaysOn>
-      <updateRate>100</updateRate>
+      <updateRate>100</updateRate>s
       <leftJoint>base_link_to_left_wheel</leftJoint>
       <rightJoint>base_link_to_right_wheel</rightJoint>
       <wheelSeparation>${wheel_separation}</wheelSeparation>
       <wheelDiameter>${wheel_diameter}</wheelDiameter>
-      <wheelTorque>2</wheelTorque>
+      <wheelTorque>200</wheelTorque>
       <commandTopic>cmd_diff_vel</commandTopic>
       <broadcastTF>false</broadcastTF>
-    </plugin>
+    </plugin> -->
   </gazebo>
 </robot>

Commit message: split up xacro file, and in process of debugging diff drive

File: swarm_ws/src/swarm_description/urdf/blackhawk_standalone.xacro (robot description, xacro)
@@ -1,19 +1,12 @@
 <?xml version="1.0"?>
 <robot name="blackhawk" xmlns:xacro="http://ros.org/wiki/xacro">
+  <!-- Values for different components of the robot-->
+  <xacro:property name="wheel_separation" value="0.02"/>
+  <xacro:property name="wheel_diameter" value="0.025"/>
+  <xacro:property name="wheel_width" value="0.005"/>
+  <xacro:property name="wheel_standoff" value="0.01"/>
+  <xacro:property name="body_length" value="0.06"/>
+  <xacro:include filename="$(find swarm_description)/urdf/macros.xacro"/>
   <link name="base_link">
-    <!-- Body geometry macro -->
-    <!-- <mesh filename="package://swarm_description/meshes/Blackhawk_resized.dae"/> -->
-    <xacro:property name="body_length" value="0.06"/>
-    <xacro:macro name="body">
-      <geometry>
-        <!--<cylinder length="${body_length}" radius="0.5" /> -->
-        <mesh filename="package://swarm_description/meshes/Blackhawk_resized.dae"/>
-      </geometry>
-    </xacro:macro>
-    <!-- Values for different components of the robot-->
-    <xacro:property name="wheel_separation" value="0.02"/>
-    <xacro:property name="wheel_diameter" value="0.025"/>
-    <xacro:property name="wheel_width" value="0.005"/>
-    <xacro:property name="wheel_standoff" value="0.01"/>
     <!-- visual -->
     <visual>
@@ -40,10 +33,4 @@
 	  <parent link="base_link"/>
   </joint>
-  <!-- Wheel geometry macro -->
-  <xacro:macro name="wheel_geometry">
-    <geometry>
-	    <cylinder length="${wheel_width}" radius="${wheel_diameter / 2}"/>
-    </geometry>
-  </xacro:macro>
   <!-- Wheel geometries -->
   <link name="left_wheel">
@@ -67,20 +54,8 @@
     </collision>
   </link>
-  <!-- Plugin to simulate driving motion -->
-  <gazebo>
-    <plugin name="gazebo_ros_control" filename="libgazebo_ros_control.so">
-      <robotSimType>gazebo_ros_control/DefaultRobotHWSim</robotSimType>
-    </plugin>
-    <!-- <plugin name="differential_drive_controller" filename="libgazebo_ros_diff_drive.so">
-      <alwaysOn>true</alwaysOn>
-      <updateRate>100</updateRate>s
-      <leftJoint>base_link_to_left_wheel</leftJoint>
-      <rightJoint>base_link_to_right_wheel</rightJoint>
-      <wheelSeparation>${wheel_separation}</wheelSeparation>
-      <wheelDiameter>${wheel_diameter}</wheelDiameter>
-      <wheelTorque>200</wheelTorque>
-      <commandTopic>cmd_diff_vel</commandTopic>
-      <broadcastTF>false</broadcastTF>
-    </plugin> -->
-  </gazebo>
+  <!-- Setting up transmissions for differential driving -->
+  <xacro:mk_transmission side="right"/>
+  <xacro:mk_transmission side="left"/>
+  <!-- Using separate file to set up Gazebo properties and plugins -->
+  <xacro:include filename="$(find swarm_description)/urdf/blackhawk_standalone.gazebo"/>
 </robot>

Commit message: Still working out diff drive errors
Differential drive attempts are throwing errors that read out to say that there is no  valid hardware interface in the joints

File: swarm_ws/src/swarm_description/urdf/blackhawk_standalone.xacro (robot description, xacro)
@@ -8,4 +8,15 @@
   <xacro:property name="body_length" value="0.06"/>
   <xacro:include filename="$(find swarm_description)/urdf/macros.xacro"/>
+  <!-- This is here to give RVIS a fixed global frame -->
+  <link name="map">
+    <visual>
+      <origin xyz="0 0 0" rpy="0 0 0"/>
+    </visual>
+  </link>
+  <joint name="map_to_base_link" type="fixed">
+    <child link="base_link"/>
+    <parent link="map"/>
+  </joint>
+  <!-- Main link for the robot_description -->
   <link name="base_link">
     <!-- visual -->
@@ -24,13 +35,4 @@
     </inertial>
   </link>
-  <!-- wheel joints -->
-  <joint name="base_link_to_left_wheel" type="fixed">
-    <child link="left_wheel" />
-    <parent link="base_link" />
-  </joint>
-  <joint name="base_link_to_right_wheel" type="fixed">
-	  <child link="right_wheel"/>
-	  <parent link="base_link"/>
-  </joint>
   <!-- Wheel geometries -->
   <link name="left_wheel">
@@ -54,7 +56,18 @@
     </collision>
   </link>
+  <!-- wheel joints -->
+  <joint name="base_link_to_left_wheel" type="fixed">
+    <child link="left_wheel" />
+    <parent link="base_link" />
+    <axis xyz="0 1 0" rpy="0 0 0"/>
+  </joint>
+  <joint name="base_link_to_right_wheel" type="fixed">
+    <child link="right_wheel"/>
+    <parent link="base_link"/>
+    <axis xyz="0 1 0" rpy="0 0 0"/>
+  </joint>
   <!-- Setting up transmissions for differential driving -->
-  <xacro:mk_transmission side="right"/>
-  <xacro:mk_transmission side="left"/>
+  <xacro:mk_transmission joint="base_link_to_right_wheel"/>
+  <xacro:mk_transmission joint="base_link_to_left_wheel"/>
   <!-- Using separate file to set up Gazebo properties and plugins -->
   <xacro:include filename="$(find swarm_description)/urdf/blackhawk_standalone.gazebo"/>

File: swarm_ws/src/swarm_description/urdf/macros.xacro (robot description, xacro)
@@ -16,11 +16,11 @@
     </xacro:macro>
     <!-- transmission macros -->
-    <xacro:macro name="mk_transmission" params="side">
-        <transmission name="${side}_wheel_transmission">
+    <xacro:macro name="mk_transmission" params="joint">
+        <transmission name="${joint}_transmission">
             <type>transmission_interface/SimpleTransmission</type>
-            <joint name="base_link_to_${side}_wheel">
-                <hardwareInteface>EffortJointInterface</hardwareInteface>
-            </joint>
-            <actuator name="${side}_wheel_actuator">
+	    <joint name="${joint}">
+		<hardwareInteface>EffortJointInterface</hardwareInteface>
+	    </joint>
+            <actuator name="${joint}_actuator">
                 <mechanicalReduction>1</mechanicalReduction>
                 <hardwareInteface>EffortJointInterface</hardwareInteface>

Commit message: updated gazebo sim

File: swarm_ws/src/swarm_description/urdf/blackhawk_standalone.xacro (robot description, xacro)
@@ -2,35 +2,36 @@
 <robot name="blackhawk" xmlns:xacro="http://ros.org/wiki/xacro">
   <!-- Values for different components of the robot-->
-  <xacro:property name="wheel_separation" value="0.02"/>
-  <xacro:property name="wheel_diameter" value="0.025"/>
+  <xacro:property name="wheel_mass" value="0.00368"/>
+  <xacro:property name="wheel_separation" value="0.018"/> <!-- side by side separation from center -->
+  <xacro:property name="wheel_diameter" value="0.028"/>
   <xacro:property name="wheel_width" value="0.005"/>
-  <xacro:property name="wheel_standoff" value="0.01"/>
-  <xacro:property name="body_length" value="0.06"/>
+  <xacro:property name="wheel_standoff" value="0.0055"/> <!-- forward/backward offset from center -->
+  <xacro:property name="body_mass" value="0.19044"/> <!-- weighed bot = 0.19784; subtract wheels (2*wheel_mass) -->
+  <xacro:property name="body_length" value="0.0766"/>
+  <xacro:property name="body_width" value="0.0697"/>
+  <xacro:property name="PI" value="3.1415926535897931"/>
   <xacro:include filename="$(find swarm_description)/urdf/macros.xacro"/>
   <!-- This is here to give RVIS a fixed global frame -->
-  <link name="map">
-    <visual>
-      <origin xyz="0 0 0" rpy="0 0 0"/>
-    </visual>
-  </link>
+  <!-- <link name="map"/>
   <joint name="map_to_base_link" type="fixed">
     <child link="base_link"/>
     <parent link="map"/>
-  </joint>
+    <origin xyz="0 0 0.0305" rpy="0 0 0"/>
+  </joint> -->
   <!-- Main link for the robot_description -->
   <link name="base_link">
     <!-- visual -->
     <visual>
-	    <origin rpy="0.0 0 0" xyz="0 0 ${body_length / 2}"/>
+      <origin xyz="0 0 0" rpy="0 0 0"/>
 	    <xacro:body/>
     </visual>
     <!-- inertial & collision -->
     <collision>
-	    <origin rpy="0.0 0 0" xyz="0 0 ${body_length / 2}"/>
+      <origin xyz="0 0 0" rpy="0 0 0"/>
         <xacro:body/>
       </collision>
     <inertial>
-      <mass value="0.05"/>
-      <inertia ixx="0.5" ixy="0.0" ixz="0.0" iyy="0.5" iyz="0.0" izz="0.5"/>
+      <origin xyz="0 0 0" rpy="0 0 0"/>
+      <xacro:body_inertial/>
     </inertial>
   </link>
@@ -38,37 +39,53 @@
   <link name="left_wheel">
     <visual>
-      <origin rpy="1.57079 0 0" xyz="${wheel_standoff} -${wheel_separation} 0"/>
+      <origin xyz="0 0 0" rpy="0 0 0"/>
       <xacro:wheel_geometry/>
+      <material name="black">
+        <color rgba="0.0 0.0 0.0 1.0"/>
+      </material>
     </visual>
     <collision>
-	    <origin rpy="1.57079 0 0" xyz="${wheel_standoff} -${wheel_separation} 0"/>
+      <origin xyz="0 0 0" rpy="0 0 0"/>
       <xacro:wheel_geometry/>
     </collision>
+    <inertial>
+      <origin xyz="0 0 0" rpy="0 0 0"/>
+      <xacro:wheel_inertial/>
+    </inertial>
   </link>
   <link name="right_wheel">
     <visual>
-      <origin rpy="-1.57079 0 0" xyz="-${wheel_standoff} ${wheel_separation} 0"/>
+      <origin xyz="0 0 0" rpy="0 0 0"/>
       <xacro:wheel_geometry/>
+      <material name="black">
+        <color rgba="0.0 0.0 0.0 1.0"/>
+      </material>
     </visual>
     <collision>
-	    <origin rpy="-1.57079 0 0" xyz="-${wheel_standoff} ${wheel_separation} 0"/>
+      <origin xyz="0 0 0" rpy="0 0 0"/>
       <xacro:wheel_geometry/>
     </collision>
+    <inertial>
+      <origin xyz="0 0 0" rpy="0 0 0"/>
+      <xacro:wheel_inertial/>
+    </inertial>
   </link>
   <!-- wheel joints -->
-  <joint name="base_link_to_left_wheel" type="fixed">
+  <joint name="base_link_to_left_wheel" type="continuous">
+    <origin xyz="${wheel_standoff} -${wheel_separation} -0.017" rpy="${PI/2} 0 0" />
     <child link="left_wheel" />
     <parent link="base_link" />
-    <axis xyz="0 1 0" rpy="0 0 0"/>
+    <axis xyz="0 0 1"/>
   </joint>
-  <joint name="base_link_to_right_wheel" type="fixed">
+  <joint name="base_link_to_right_wheel" type="continuous">
+    <origin xyz="-${wheel_standoff} ${wheel_separation} -0.017" rpy="-${PI/2} 0 0" />
     <child link="right_wheel"/>
     <parent link="base_link"/>
-    <axis xyz="0 1 0" rpy="0 0 0"/>
+    <axis xyz="0 0 1"/>
   </joint>
+  <!-- Using separate file to set up Gazebo properties and plugins -->
+  <xacro:include filename="$(find swarm_description)/urdf/blackhawk_standalone.gazebo"/>
   <!-- Setting up transmissions for differential driving -->
   <xacro:mk_transmission joint="base_link_to_right_wheel"/>
   <xacro:mk_transmission joint="base_link_to_left_wheel"/>
-  <!-- Using separate file to set up Gazebo properties and plugins -->
-  <xacro:include filename="$(find swarm_description)/urdf/blackhawk_standalone.gazebo"/>
 </robot>

File: swarm_ws/src/swarm_description/urdf/macros.xacro (robot description, xacro)
@@ -1,30 +1,41 @@
 <?xml version="1.0"?>
 <robot name="blackhawk" xmlns:xacro="http://ros.org/wiki/xacro">
-    <!-- Body geometry macro -->
-    <!-- <mesh filename="package://swarm_description/meshes/Blackhawk_resized.dae"/> -->
-    <xacro:macro name="body">
-      <geometry>
-        <!--<cylinder length="${body_length}" radius="0.5" /> -->
-        <mesh filename="package://swarm_description/meshes/Blackhawk_resized.dae"/>
-      </geometry>
-    </xacro:macro>
-    <!-- Wheel geometry macro -->
-    <xacro:macro name="wheel_geometry">
-        <geometry>
-            <cylinder length="${wheel_width}" radius="${wheel_diameter / 2}"/>
-        </geometry>
-    </xacro:macro>
-    <!-- transmission macros -->
-    <xacro:macro name="mk_transmission" params="joint">
-        <transmission name="${joint}_transmission">
-            <type>transmission_interface/SimpleTransmission</type>
-	    <joint name="${joint}">
-		<hardwareInteface>EffortJointInterface</hardwareInteface>
-	    </joint>
-            <actuator name="${joint}_actuator">
-                <mechanicalReduction>1</mechanicalReduction>
-                <hardwareInteface>EffortJointInterface</hardwareInteface>
-            </actuator>
-        </transmission>
-    </xacro:macro>
+  <!-- Body geometry macro -->
+  <xacro:macro name="body">
+    <geometry>
+      <!-- <cylinder length="${body_length}" radius="0.035" /> -->
+      <mesh filename="package://swarm_description/meshes/Blackhawk_Full_resized.dae"/>
+    </geometry>
+  </xacro:macro>
+  <xacro:macro name="body_inertial">
+    <mass value="${body_mass}"/>
+    <inertia ixx="0.000150942" ixy="0.0" ixz="0.0" iyy="0.000150942" iyz="0.0" izz="0.000115647"/>
+  </xacro:macro>
+  <!-- Wheel geometry macro -->
+  <xacro:macro name="wheel_geometry">
+    <geometry>
+      <cylinder length="${wheel_width}" radius="${wheel_diameter / 2}"/>
+    </geometry>
+  </xacro:macro>
+  <xacro:macro name="wheel_inertial">
+    <mass value="${wheel_mass}" />
+    <inertia ixx="1.88e-7"   ixy="0"     ixz="0"
+                          iyy="1.88e-7"  iyz="0"
+                                      izz="3.61e-7" />
+  </xacro:macro>
+  <!-- transmission macros -->
+  <xacro:macro name="mk_transmission" params="joint">
+    <transmission name="${joint}_transmission">
+      <type>transmission_interface/SimpleTransmission</type>
+      <joint name="${joint}">
+        <hardwareInterface>hardware_interface/EffortJointInterface</hardwareInterface>
+        <!-- <hardwareInterface>hardware_interface/VelocityJointInterface</hardwareInterface> -->
+      </joint>
+      <actuator name="${joint}_actuator">
+        <mechanicalReduction>1</mechanicalReduction>
+        <hardwareInterface>hardware_interface/EffortJointInterface</hardwareInterface>
+        <!-- <hardwareInterface>hardware_interface/VelocityJointInterface</hardwareInterface> -->
+      </actuator>
+    </transmission>
+  </xacro:macro>
 </robot>
